Commit message: hector_quadrotor_urdf: cleaned up urdf descriptions

File: hector_quadrotor_controller/urdf/model_based_navigation.urdf.xacro (robot description, xacro)
@@ -1,7 +1,4 @@
 <?xml version="1.0"?>
-<robot
-xmlns:controller="http://playerstage.sourceforge.net/gazebo/xmlschema/#controller"
-xmlns:xacro="http://ros.org/wiki/xacro"
->
+<robot xmlns:xacro="http://ros.org/wiki/xacro">
   <!-- Quadrotor Model Based Navigation Plugin -->
   <xacro:macro name="model_based_navigation">

File: hector_quadrotor_controller/urdf/quadrotor_pose_estimation.urdf.xacro (robot description, xacro)
@@ -1,5 +1,4 @@
 <?xml version="1.0"?>
 <robot
-xmlns:controller="http://playerstage.sourceforge.net/gazebo/xmlschema/#controller"
 xmlns:xacro="http://ros.org/wiki/xacro"
 >

File: hector_quadrotor_urdf/urdf/quadrotor.urdf.xacro (robot description, xacro)
@@ -1,11 +1,10 @@
 <?xml version="1.0"?>
-<robot name="quadrotor"
-    xmlns:sensor="http://playerstage.sourceforge.net/gazebo/xmlschema/#sensor"
-    xmlns:controller="http://playerstage.sourceforge.net/gazebo/xmlschema/#controller"
-    xmlns:interface="http://playerstage.sourceforge.net/gazebo/xmlschema/#interface"
-    xmlns:xacro="http://playerstage.sourceforge.net/gazebo/xmlschema/#interface">
+<robot
+  name="quadrotor"
+  xmlns:xacro="http://ros.org/wiki/xacro"
+>
     <!-- Included URDF Files -->
-    <include filename="$(find hector_quadrotor_urdf)/urdf/quadrotor_base.urdf.xacro" />
+    <xacro:include filename="$(find hector_quadrotor_urdf)/urdf/quadrotor_base.urdf.xacro" />
     <!-- Instantiate quadrotor_base_macro once (has no parameters atm) -->
-    <quadrotor_base_macro />
+    <xacro:quadrotor_base_macro />
 </robot>

File: hector_quadrotor_urdf/urdf/quadrotor_base.urdf.xacro (robot description, xacro)
@@ -1,11 +1,7 @@
 <?xml version="1.0"?>
-<robot xmlns:sensor="http://playerstage.sourceforge.net/gazebo/xmlschema/#sensor"
-xmlns:controller="http://playerstage.sourceforge.net/gazebo/xmlschema/#controller"
-xmlns:interface="http://playerstage.sourceforge.net/gazebo/xmlschema/#interface"
-xmlns:xacro="http://ros.org/wiki/xacro"
->
-  <include filename="$(find hector_sensors_description)/urdf/sonar_sensor.urdf.xacro" />
-  <include filename="$(find hector_quadrotor_gazebo)/urdf/quadrotor_plugins.urdf.xacro" />
-  <property name="pi" value="3.1415926535897931" />
+<robot xmlns:xacro="http://ros.org/wiki/xacro">
+  <xacro:include filename="$(find hector_sensors_description)/urdf/sonar_sensor.urdf.xacro" />
+  <xacro:include filename="$(find hector_quadrotor_gazebo)/urdf/quadrotor_plugins.urdf.xacro" />
+  <xacro:property name="pi" value="3.1415926535897931" />
   <!-- Main quadrotor link -->
   <xacro:macro name="quadrotor_base_macro">
@@ -30,12 +26,12 @@
     </link>
     <!-- Sonar height sensor -->
-    <sonar_sensor name="sonar" parent="base_link" ros_topic="sonar_height" update_rate="10" min_range="0.03" max_range="3.0" field_of_view="${40*pi/180}" ray_count="3">
+    <xacro:sonar_sensor name="sonar" parent="base_link" ros_topic="sonar_height" update_rate="10" min_range="0.03" max_range="3.0" field_of_view="${40*pi/180}" ray_count="3">
       <origin xyz="-0.16 0.0 -0.012" rpy="0 ${90*pi/180} 0"/>
-    </sonar_sensor>
+    </xacro:sonar_sensor>
     <gazebo reference="base_link">
       <turnGravityOff>false</turnGravityOff>
     </gazebo>
     <!-- Gazebo Plugins -->
-    <quadrotor_plugins/>
+    <xacro:quadrotor_plugins/>
   </xacro:macro>
 </robot>

File: hector_quadrotor_urdf/urdf/quadrotor_downward_cam.urdf.xacro (robot description, xacro)
@@ -1,20 +1,19 @@
 <?xml version="1.0"?>
-<robot name="quadrotor_hokuyo_utm30lx"
-xmlns:sensor="http://playerstage.sourceforge.net/gazebo/xmlschema/#sensor"
-xmlns:controller="http://playerstage.sourceforge.net/gazebo/xmlschema/#controller"
-xmlns:interface="http://playerstage.sourceforge.net/gazebo/xmlschema/#interface"
-xmlns:xacro="http://playerstage.sourceforge.net/gazebo/xmlschema/#interface">
-    <property name="M_PI" value="3.1415926535897931" />
+<robot
+  name="quadrotor"
+  xmlns:xacro="http://ros.org/wiki/xacro"
+>
+    <xacro:property name="M_PI" value="3.1415926535897931" />
     <!-- Included URDF Files -->
-    <include filename="$(find hector_quadrotor_urdf)/urdf/quadrotor_base.urdf.xacro" />
+    <xacro:include filename="$(find hector_quadrotor_urdf)/urdf/quadrotor_base.urdf.xacro" />
     <!-- Instantiate quadrotor_base_macro once (has no parameters atm) -->
-    <quadrotor_base_macro />
+    <xacro:quadrotor_base_macro />
     <!-- Hokuyo UTM-30LX mounted upside down below the quadrotor body -->
-<!--    <include filename="$(find hector_sensors_description)/urdf/hokuyo_utm30lx.urdf.xacro" />
+<!--    <xacro:include filename="$(find hector_sensors_description)/urdf/hokuyo_utm30lx.urdf.xacro" />
     <xacro:hokuyo_utm30lx name="laser0" parent="base_link" ros_topic="scan" update_rate="40" ray_count="1081" min_angle="135" max_angle="-135">
       <origin xyz="0.0 0.0 -0.097" rpy="${M_PI} 0 0"/>
     </xacro:hokuyo_utm30lx>-->
     <!-- Downward facing camera -->
-    <include filename="$(find hector_sensors_description)/urdf/generic_camera.urdf.xacro" />
+    <xacro:include filename="$(find hector_sensors_description)/urdf/generic_camera.urdf.xacro" />
     <xacro:generic_camera name="downward_cam" parent="base_link" ros_topic="camera/image" cam_info_topic="camera/camera_info" update_rate="20" res_x="640" res_y="480" image_format="L8" hfov="100">
       <origin xyz="0.4 0.0 -0.0" rpy="0 ${M_PI/2} 0"/>

File: hector_quadrotor_urdf/urdf/quadrotor_hokuyo_utm30lx.urdf.xacro (robot description, xacro)
@@ -1,20 +1,19 @@
 <?xml version="1.0"?>
-<robot name="quadrotor_hokuyo_utm30lx"
-xmlns:sensor="http://playerstage.sourceforge.net/gazebo/xmlschema/#sensor"
-xmlns:controller="http://playerstage.sourceforge.net/gazebo/xmlschema/#controller"
-xmlns:interface="http://playerstage.sourceforge.net/gazebo/xmlschema/#interface"
-xmlns:xacro="http://playerstage.sourceforge.net/gazebo/xmlschema/#interface">
-    <property name="M_PI" value="3.1415926535897931" />
+<robot
+  name="quadrotor"
+  xmlns:xacro="http://ros.org/wiki/xacro"
+>
+    <xacro:property name="M_PI" value="3.1415926535897931" />
     <!-- Included URDF Files -->
-    <include filename="$(find hector_quadrotor_urdf)/urdf/quadrotor_base.urdf.xacro" />
+    <xacro:include filename="$(find hector_quadrotor_urdf)/urdf/quadrotor_base.urdf.xacro" />
     <!-- Instantiate quadrotor_base_macro once (has no parameters atm) -->
-    <quadrotor_base_macro />
+    <xacro:quadrotor_base_macro />
     <!-- Hokuyo UTM-30LX mounted upside down below the quadrotor body -->
-    <include filename="$(find hector_sensors_description)/urdf/hokuyo_utm30lx.urdf.xacro" />
+    <xacro:include filename="$(find hector_sensors_description)/urdf/hokuyo_utm30lx.urdf.xacro" />
     <xacro:hokuyo_utm30lx name="laser0" parent="base_link" ros_topic="scan" update_rate="40" ray_count="1081" min_angle="135" max_angle="-135">
       <origin xyz="0.0 0.0 -0.097" rpy="${M_PI} 0 0"/>
     </xacro:hokuyo_utm30lx>
     <!-- Forward facing camera -->
-    <include filename="$(find hector_sensors_description)/urdf/generic_camera.urdf.xacro" />
+    <xacro:include filename="$(find hector_sensors_description)/urdf/generic_camera.urdf.xacro" />
     <xacro:generic_camera name="front_cam" parent="base_link" ros_topic="camera/image" cam_info_topic="camera/camera_info" update_rate="10" res_x="320" res_y="240" image_format="R8G8B8" hfov="90">
       <origin xyz="0.05 0.0 -0.06" rpy="0 0 0"/>

File: hector_quadrotor_urdf/urdf/quadrotor_with_asus.urdf.xacro (robot description, xacro)
@@ -1,15 +1,14 @@
 <?xml version="1.0"?>
-<robot name="quadrotor_asus_xiton_pro_live"
-xmlns:sensor="http://playerstage.sourceforge.net/gazebo/xmlschema/#sensor"
-xmlns:controller="http://playerstage.sourceforge.net/gazebo/xmlschema/#controller"
-xmlns:interface="http://playerstage.sourceforge.net/gazebo/xmlschema/#interface"
-xmlns:xacro="http://playerstage.sourceforge.net/gazebo/xmlschema/#interface">
-    <property name="M_PI" value="3.1415926535897931" />
+<robot
+  name="quadrotor"
+  xmlns:xacro="http://ros.org/wiki/xacro"
+>
+    <xacro:property name="M_PI" value="3.1415926535897931" />
     <!-- Included URDF Files -->
-    <include filename="$(find hector_quadrotor_urdf)/urdf/quadrotor_base.urdf.xacro" />
+    <xacro:include filename="$(find hector_quadrotor_urdf)/urdf/quadrotor_base.urdf.xacro" />
     <!-- Instantiate quadrotor_base_macro once (has no parameters atm) -->
-    <quadrotor_base_macro />
+    <xacro:quadrotor_base_macro />
     <!-- Asus Xiton Live Pro -->
-    <include filename="$(find hector_sensors_description)/urdf/asus_camera.urdf.xacro" />
+    <xacro:include filename="$(find hector_sensors_description)/urdf/asus_camera.urdf.xacro" />
     <xacro:asus_camera name="camera" parent="base_link">
       <origin xyz="0.1 0.0 -0.03" rpy="0 ${M_PI/9} 0"/>

File: hector_quadrotor_urdf/urdf/quadrotor_with_asus_with_hokuyo_utm30lx.urdf.xacro (robot description, xacro)
@@ -1,20 +1,19 @@
 <?xml version="1.0"?>
-<robot name="quadrotor_with_asus_xiton_pro_live_with_hokuyo_utm30lx"
-xmlns:sensor="http://playerstage.sourceforge.net/gazebo/xmlschema/#sensor"
-xmlns:controller="http://playerstage.sourceforge.net/gazebo/xmlschema/#controller"
-xmlns:interface="http://playerstage.sourceforge.net/gazebo/xmlschema/#interface"
-xmlns:xacro="http://playerstage.sourceforge.net/gazebo/xmlschema/#interface">
-    <property name="M_PI" value="3.1415926535897931" />
+<robot
+  name="quadrotor"
+  xmlns:xacro="http://ros.org/wiki/xacro"
+>
+    <xacro:property name="M_PI" value="3.1415926535897931" />
     <!-- Included URDF Files -->
-    <include filename="$(find hector_quadrotor_urdf)/urdf/quadrotor_base.urdf.xacro" />
+    <xacro:include filename="$(find hector_quadrotor_urdf)/urdf/quadrotor_base.urdf.xacro" />
     <!-- Instantiate quadrotor_base_macro once (has no parameters atm) -->
-    <quadrotor_base_macro />
+    <xacro:quadrotor_base_macro />
     <!-- Hokuyo UTM-30LX mounted upside down below the quadrotor body -->
-    <include filename="$(find hector_sensors_description)/urdf/hokuyo_utm30lx.urdf.xacro" />
+    <xacro:include filename="$(find hector_sensors_description)/urdf/hokuyo_utm30lx.urdf.xacro" />
     <xacro:hokuyo_utm30lx name="laser0" parent="base_link" ros_topic="scan" update_rate="40" ray_count="1081" min_angle="135" max_angle="-135">
       <origin xyz="0.0 0.0 -0.097" rpy="${M_PI} 0 0"/>
     </xacro:hokuyo_utm30lx>
     <!-- Asus Xiton Live Pro -->
-    <include filename="$(find hector_sensors_description)/urdf/asus_camera.urdf.xacro" />
+    <xacro:include filename="$(find hector_sensors_description)/urdf/asus_camera.urdf.xacro" />
     <xacro:asus_camera name="camera" parent="base_link">
       <origin xyz="0.1 0.0 -0.03" rpy="0 ${M_PI/9} 0"/>

File: hector_quadrotor_urdf/urdf/quadrotor_with_cam.urdf.xacro (robot description, xacro)
@@ -1,20 +1,19 @@
 <?xml version="1.0"?>
-<robot name="quadrotor_hokuyo_utm30lx"
-xmlns:sensor="http://playerstage.sourceforge.net/gazebo/xmlschema/#sensor"
-xmlns:controller="http://playerstage.sourceforge.net/gazebo/xmlschema/#controller"
-xmlns:interface="http://playerstage.sourceforge.net/gazebo/xmlschema/#interface"
-xmlns:xacro="http://playerstage.sourceforge.net/gazebo/xmlschema/#interface">
-    <property name="M_PI" value="3.1415926535897931" />
+<robot
+  name="quadrotor"
+  xmlns:xacro="http://ros.org/wiki/xacro"
+>
+    <xacro:property name="M_PI" value="3.1415926535897931" />
     <!-- Included URDF Files -->
-    <include filename="$(find hector_quadrotor_urdf)/urdf/quadrotor_base.urdf.xacro" />
+    <xacro:include filename="$(find hector_quadrotor_urdf)/urdf/quadrotor_base.urdf.xacro" />
     <!-- Instantiate quadrotor_base_macro once (has no parameters atm) -->
-    <quadrotor_base_macro />
+    <xacro:quadrotor_base_macro />
     <!-- Hokuyo UTM-30LX mounted upside down below the quadrotor body -->
-    <!-- include filename="$(find hector_sensors_description)/urdf/hokuyo_utm30lx.urdf.xacro" />
+    <!-- xacro:include filename="$(find hector_sensors_description)/urdf/hokuyo_utm30lx.urdf.xacro" />
     <xacro:hokuyo_utm30lx name="laser0" parent="base_link" ros_topic="scan" update_rate="40" ray_count="1081" min_angle="135" max_angle="-135">
       <origin xyz="0.0 0.0 -0.097" rpy="${M_PI} 0 0"/>
     </xacro:hokuyo_utm30lx -->
     <!-- Forward facing camera -->
-    <include filename="$(find hector_sensors_description)/urdf/generic_camera.urdf.xacro" />
+    <xacro:include filename="$(find hector_sensors_description)/urdf/generic_camera.urdf.xacro" />
     <xacro:generic_camera name="front_cam" parent="base_link" ros_topic="camera/image" cam_info_topic="camera/camera_info" update_rate="10" res_x="320" res_y="240" image_format="R8G8B8" hfov="90">
       <origin xyz="0.05 0.0 -0.06" rpy="0 0 0"/>

File: hector_quadrotor_urdf/urdf/quadrotor_with_kinect.urdf.xacro (robot description, xacro)
@@ -1,15 +1,14 @@
 <?xml version="1.0"?>
-<robot name="quadrotor_hokuyo_utm30lx"
-xmlns:sensor="http://playerstage.sourceforge.net/gazebo/xmlschema/#sensor"
-xmlns:controller="http://playerstage.sourceforge.net/gazebo/xmlschema/#controller"
-xmlns:interface="http://playerstage.sourceforge.net/gazebo/xmlschema/#interface"
-xmlns:xacro="http://playerstage.sourceforge.net/gazebo/xmlschema/#interface">
-    <property name="M_PI" value="3.1415926535897931" />
+<robot
+  name="quadrotor"
+  xmlns:xacro="http://ros.org/wiki/xacro"
+>
+    <xacro:property name="M_PI" value="3.1415926535897931" />
     <!-- Included URDF Files -->
-    <include filename="$(find hector_quadrotor_urdf)/urdf/quadrotor_base.urdf.xacro" />
+    <xacro:include filename="$(find hector_quadrotor_urdf)/urdf/quadrotor_base.urdf.xacro" />
     <!-- Instantiate quadrotor_base_macro once (has no parameters atm) -->
-    <quadrotor_base_macro />
+    <xacro:quadrotor_base_macro />
     <!-- Kinect -->
-    <include filename="$(find hector_sensors_description)/urdf/kinect_camera.urdf.xacro" />
+    <xacro:include filename="$(find hector_sensors_description)/urdf/kinect_camera.urdf.xacro" />
     <xacro:kinect_camera name="camera" parent="base_link">
       <origin xyz="0.05 0.0 -0.06" rpy="0 0 0"/>
